File: Macropad.kicad_pcb (KiCad board)
At the start: 2 copper layers, 96.5 x 96.5 mm, 94 parts, among them Q1 Q_NPN_BCE, U1 ARDUINO_PRO_MICRO

Commit message: _
Other:
- board text added: "JLCJLCJLCJLC"
Changed lines of the file:
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@@
   (general
     (thickness 1.6)
-    (drawings 10)
+    (drawings 11)
     (tracks 1001)
     (zones 0)
@@
       (net 73 RST))
   )
+  (gr_text JLCJLCJLCJLC (at 71.74484 36.02228 90) (layer B.SilkS)
+    (effects (font (size 0.9 0.9) (thickness 0.2)))
+  )
   (gr_text "Rev 1.0" (at 66.548 112.395) (layer B.SilkS)
